Commit message: 3090: spotr and baseline train, sample grasp point in full scene; modify sim environment camera pose and board size;

File: experiment/resources/board.urdf (robot description, URDF)
Before this commit: robot board, 1 links, 0 joints
Links:
- link base_link: geometry collision box size=0.6 0.6 0.01; visual box size=0.6 0.6 0.01

Commit message: collect vis result: sim, add 3d model. backbone: key point. test_scene, grasp pose.

File: experiment/resources/board.urdf (robot description, URDF)
Before this commit: robot board, 1 links, 0 joints
Links:
- link base_link: geometry collision box size=0.80 0.80 0.005; visual box size=0.80 0.80 0.005
